File: MeshMite.kicad_pcb (KiCad board)
At the start: 4 copper layers, 27.5 x 67.5 mm, 27 parts, among them J1 DX07S024XA8R700, J3 ANT, U1 nRF52840, U2 Wio-SX1262, U3 BQ25504, U4 TP4056-42-ESOP8

Commit message: modularize
Parts:
- removed 0.1uF1, C5, C6: C, Capacitor_SMD:C_0402_1005Metric
- removed 15.52M1, 4.4M1, R1, R2, R3: R, Resistor_SMD:R_0201_0603Metric
- removed BT1: >= 100 uF, Connector_JST:JST_EH_B2B-EH-A_1x02_P2.50mm_Vertical
- removed C7: 4.7 uF, Capacitor_SMD:C_0805_2012Metric
- removed C8: 0.1 uF, Capacitor_SMD:C_0402_1005Metric
- removed C9: 10 uF, Capacitor_SMD:C_0805_2012Metric
- removed J1: DX07S024XA8R700, DX07S024XA8R700:JAE_DX07S024XA8R700
- removed J3: ANT, Connector_Coaxial:SMA_Amphenol_132289_EdgeMount
- removed L2: 0, Inductor_SMD:L_0201_0603Metric
- removed R4, R5: 5.1k, Resistor_SMD:R_0201_0603Metric
- removed SC1: Solar_Cell, Connector_JST:JST_EH_B2B-EH-A_1x02_P2.50mm_Vertical
- removed U1: nRF52840, Package_DFN_QFN:QFN-48-1EP_6x6mm_P0.4mm_EP4.6x4.6mm
- removed U2: Wio-SX1262, Wio-SX1262:Wio-SX11262_footprint
- added C11: 100 pF, Capacitor_SMD:C_0805_2012Metric, F.Cu at (106.3, 71.4)
- added C12: 100 nF, Capacitor_SMD:C_0402_1005Metric, F.Cu at (110.1, 65.2)
- added J2: Conn_ARM_JTAG_SWD_10, Connector_PinHeader_1.27mm:PinHeader_2x05_P1.27mm_Vertical, F.Cu at (110.8, 67.9)
- added L4: 10 uH, Inductor_SMD:L_0805_2012Metric, F.Cu at (110.9, 76.0)
- C1: value 4.7 uF -> 100 nF; footprint Capacitor_SMD:C_0805_2012Metric -> Capacitor_SMD:C_0402_1005Metric
- C2: value 0.1 uF -> 47 nF
- C3: value 4.7 uF -> 1.0 uF; footprint Capacitor_SMD:C_0805_2012Metric -> Capacitor_SMD:C_0402_1005Metric
- C4: value 0.1 uF -> 100 nF
- L1: value L -> 15 nH
- U3: value BQ25504 -> nRF52840; footprint Package_DFN_QFN:VQFN-16-1EP_3x3mm_P0.5mm_EP1.68x1.68mm -> Package_DFN_QFN:QFN-48-1EP_6x6mm_P0.4mm_EP4.6x4.6mm
- U4: value TP4056-42-ESOP8 -> Wio-SX1262; footprint Package_SO:SOIC-8-1EP_3.9x4.9mm_P1.27mm_EP2.41x3.3mm_ThermalVias -> Wio-SX1262:Wio-SX11262_footprint
- moved C1 67.6 mm to (110.1, 57.4), turned to 0 degrees
- moved U4 62.4 mm to (96.2, 68.6), turned to 0 degrees
- moved C4 60.8 mm to (110.1, 63.3), turned to 0 degrees
- moved L1 58.2 mm to (105.3, 73.8)
- moved C2 57.4 mm to (110.1, 59.3), turned to 0 degrees
- moved C3 55.2 mm to (110.1, 61.3), turned to 0 degrees
- moved U3 45.8 mm to (99.9, 74.0)
Connections:
- C1 pad 2: Net-(SC1--) -> Net-(U3-DEC1)
- C2 pad 1: Net-(U3-VSTOR) -> GND
- C2 pad 2: +3V3 -> GND
- C3 pad 1: Net-(U3-VSTOR) -> GND
- C3 pad 2: +3V3 -> GND
- C4 pad 1: GND -> +3V3
- C4 pad 2: Net-(U3-OT_PROG) -> GND
- L1 pad 1: Net-(SC1--) -> Net-(L1-Pad1)
- L1 pad 2: Net-(U3-LBST) -> GND
- U3 pad 1: GND -> Net-(U3-DEC1)
- U3 pad 10: unconnected-(U3-OK_PROG-Pad10) -> /LORA_BUSY
- U3 pad 11: unconnected-(U3-VBAT_OK-Pad11) -> /LORA_DIO
- U3 pad 12: GND -> +3V3
- U3 pad 13: GND -> unconnected-(U3-P0.13-Pad13)
- U3 pad 14: VBAT -> unconnected-(U3-P0.14-Pad14)
- U3 pad 15: Net-(U3-VSTOR) -> unconnected-(U3-P0.17-Pad15)
- U3 pad 16: Net-(U3-LBST) -> /RESET
- U3 pad 2: Net-(SC1--) -> unconnected-(U3-P0.00-Pad2)
- U3 pad 3: Net-(U3-VOC_SAMP) -> unconnected-(U3-P0.01-Pad3)
- U3 pad 4: unconnected-(U3-VREF_SAMP-Pad4) -> /LORA_NSS
- U3 pad 5: Net-(U3-OT_PROG) -> /LORA_NRST
- U3 pad 6: Net-(U3-VBAT_OV) -> /LORA_SCK
- U3 pad 7: Net-(U3-VRDIV) -> /LORA_MOSI
- U3 pad 8: Net-(U3-VBAT_OV) -> /LORA_MISO
- U3 pad 9: GND -> /LORA_RF_SW
- U4 pad 1: GND -> /LORA_RF_SW
- U4 pad 2: GND -> /LORA_MISO
- U4 pad 3: GND -> /LORA_MOSI
- U4 pad 4: Net-(J1-VBUS_A1) -> /LORA_SCK
- U4 pad 5: VBAT -> /LORA_NRST
- U4 pad 6: GND -> /LORA_NSS
- U4 pad 8: GND -> +3V3
- U4 pad 9: GND -> unconnected-(U4-ANT-Pad9)
Routing:
- net D-: track 34.1 -> 0.00 mm
- net D+: track 26.0 -> 0.00 mm
- net /nrf52/LORA_BUSY: track 19.9 -> 0.00 mm
- net /nrf52/LORA_DIO: track 19.8 -> 0.00 mm
- net GND: track 19.6 -> 0.00 mm, vias 8 -> 0
- net Net-(J1-VBUS_A1): track 12.5 -> 0.00 mm, vias 1 -> 0
- net VBAT: track 11.9 -> 0.00 mm, vias 2 -> 0
- net Net-(SC1--): track 8.81 -> 0.00 mm
- net +3V3: track 8.30 -> 0.00 mm, vias 3 -> 0
- net /nrf52/LORA_RF_SW: track 7.53 -> 0.00 mm
- net /nrf52/LORA_MISO: track 7.17 -> 0.00 mm
- net /nrf52/LORA_MOSI: track 6.81 -> 0.00 mm
- net /nrf52/LORA_SCK: track 6.44 -> 0.00 mm
- net /nrf52/LORA_NRST: track 6.08 -> 0.00 mm
- net /nrf52/LORA_NSS: track 6.04 -> 0.00 mm
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- removed copper zone on In1.Cu, net GND
Other:
- board outline removed
