File: MeshMite.kicad_sch (KiCad schematic)
At the start: 0 parts

Commit message: modularize
Parts:
- added C1, C12, C4, C6, C7, C8, C9: 100 nF, Capacitor_SMD:C_0402_1005Metric, symbol Device:C
- added C11: 100 pF, Capacitor_SMD:C_0805_2012Metric, symbol Device:C
- added C2: 47 nF, Capacitor_SMD:C_0402_1005Metric, symbol Device:C
- added C3: 1.0 uF, Capacitor_SMD:C_0402_1005Metric, symbol Device:C
- added C5: 47 uF, JLCImport:EEE-FT1H470AP, symbol Device:C
- added J1: JST, Connector_JST:JST_EH_B4B-EH-A_1x04_P2.50mm_Vertical, symbol Connector:Conn_01x04_Pin
- added J2: Conn_ARM_JTAG_SWD_10, Connector_PinHeader_1.27mm:PinHeader_2x05_P1.27mm_Vertical, symbol Connector:Conn_ARM_JTAG_SWD_10
- added L1: 15 nH, Inductor_SMD:L_0201_0603Metric, symbol Device:L
- added L4: 10 uH, Inductor_SMD:L_0805_2012Metric, symbol Device:L
- added TP1, TP2, TP3: TestPoint, TestPoint:TestPoint_Pad_1.0x1.0mm, symbol Connector:TestPoint
- added U3: nRF52840, Package_DFN_QFN:QFN-48-1EP_6x6mm_P0.4mm_EP4.6x4.6mm, symbol MCU_Nordic:nRF52840
- added U4: Wio-SX1262, Wio-SX1262:Wio-SX11262_footprint, symbol Wio-SX1262:libdb_Module/114993390
Connections:
- new net: C1.2, U3.1 (DEC1)
- new net: L4.1, U3.47 (DCC)
- new net: L1.1, L4.2
- new net +3V3: C12.2, C4.1, C5.1, C6.1, C7.1, C8.1, C9.1, J1.1 (Pin_1), J2.1 (VTref), TP2.1, TP3.1, U3.12 (VDD), U3.17 (VDD), U3.25 (VDD), U3.37 (VDD), U3.48 (VDD), U4.8 (VCC)
- new net GND: C1.1, C11.1, C11.2, C12.1, C2.1, C2.2, C3.1, C3.2, C4.2, C5.2, C6.2, C7.2, C8.2, C9.2, J1.2 (Pin_2), J1.3 (Pin_3), J2.3 (GND), J2.5 (GND), J2.9 (GNDDetect), L1.2, TP1.1, U3.33 (DEC6), U3.45 (VSS), U3.46 (DEC4), U3.49 (VSS), U4.7 (GND1)
- new net LORA_BUSY: U3.10 (P0.11), U4.11 (BUSY)
- new net LORA_DIO: U3.11 (P0.12), U4.12 (DIO1)
- new net LORA_MISO: U3.8 (P1.08), U4.2 (MISO)
- new net LORA_MOSI: U3.7 (P0.08), U4.3 (MOSI)
- new net LORA_NRST: U3.5 (P0.05), U4.5 (RST)
- new net LORA_NSS: U3.4 (P0.04), U4.6 (NSS)
- new net LORA_RF_SW: U3.9 (P1.09), U4.1 (RF_SW1)
- new net LORA_SCK: U3.6 (P0.07), U4.4 (SCK)
- new net RESET: J2.10 (~{RESET}), U3.16 (P0.18)
- new net SWCLK: J2.4 (SWCLK/TCK), U3.27 (SWDCLK)
- new net SWDIO: J2.2 (SWDIO/TMS), U3.26 (SWDIO)
- no-connect marks 0 -> 8
Other:
- removed sheet nrf52
- removed sheet peripherals
