File: _autosave-MeshMite.kicad_pcb (KiCad board)
At the start: 4 copper layers, 22 parts, among them J1 ANT, J2 Conn_ARM_SWD_TagConnect_TC203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, U4 nRF52840, U5 Wio-SX1262, U6 BQ25504

Commit message: modularize
Parts:
- removed 0.1uF2, C10: C, Capacitor_SMD:C_0402_1005Metric
- removed 15.52M2, 4.4M2, R4, R5, R6: R, Resistor_SMD:R_0201_0603Metric
- removed BT2: >= 100 uF, Connector_JST:JST_EH_B2B-EH-A_1x02_P2.50mm_Vertical
- removed C13: 0.1 uF, Capacitor_SMD:C_0402_1005Metric
- removed C14: 4.7 uF, Capacitor_SMD:C_0805_2012Metric
- removed L3: 0, Inductor_SMD:L_0201_0603Metric
- removed SC2: Solar_Cell, Connector_JST:JST_EH_B2B-EH-A_1x02_P2.50mm_Vertical
- removed U5: Wio-SX1262, Wio-SX1262:Wio-SX11262_footprint
- removed U6: BQ25504, Package_DFN_QFN:VQFN-16-1EP_3x3mm_P0.5mm_EP1.68x1.68mm
- added C1: 100 nF, Capacitor_SMD:C_0402_1005Metric, F.Cu at (97.0, 63.0)
- added C2: 47 nF, Capacitor_SMD:C_0402_1005Metric, F.Cu at (99.6, 66.6)
- added C3: 1.0 uF, Capacitor_SMD:C_0402_1005Metric, F.Cu at (98.4, 66.6)
- added C4: 100 nF, Capacitor_SMD:C_0402_1005Metric, F.Cu at (98.5, 69.3)
- added C5: 47 uF, JLCImport:EEE-FT1H470AP, F.Cu at (91.3, 79.0)
- added C6: 100 nF, Capacitor_SMD:C_0402_1005Metric, F.Cu at (98.2, 64.0)
- added C8: 100 nF, Capacitor_SMD:C_0402_1005Metric, F.Cu at (90.8, 63.5)
- added L1: 15 nH, Inductor_SMD:L_0201_0603Metric, F.Cu at (101.0, 66.0)
- added U3: nRF52840, Package_DFN_QFN:QFN-48-1EP_6x6mm_P0.4mm_EP4.6x4.6mm, F.Cu at (94.0, 67.8)
- C11: value 0.1 uF -> 100 pF; footprint Capacitor_SMD:C_0402_1005Metric -> Capacitor_SMD:C_0805_2012Metric
- C12: value 4.7 uF -> 100 nF; footprint Capacitor_SMD:C_0805_2012Metric -> Capacitor_SMD:C_0402_1005Metric
- C7: value 0.1 uF -> 100 nF
- C9: value C -> 100 nF
- J1: value ANT -> JST; footprint Connector_Coaxial:SMA_Amphenol_132289_EdgeMount -> Connector_JST:JST_EH_B4B-EH-A_1x04_P2.50mm_Vertical
- J2: value Conn_ARM_SWD_TagConnect_TC2030-NL -> Conn_ARM_JTAG_SWD_10; footprint Connector:Tag-Connect_TC2030-IDC-NL_2x03_P1.27mm_Vertical -> Connector_PinHeader_1.27mm:PinHeader_2x05_P1.27mm_Vertical
- L4: value L -> 10 uH; footprint Inductor_SMD:L_0201_0603Metric -> Inductor_SMD:L_0805_2012Metric
- U4: value nRF52840 -> Wio-SX1262; footprint Package_DFN_QFN:QFN-48-1EP_6x6mm_P0.4mm_EP4.6x4.6mm -> Wio-SX1262:Wio-SX11262_footprint
- moved L4 56.4 mm to (100.9, 64.4)
- moved J1 49.9 mm to (90.0, 86.0), turned to 0 degrees
- moved C11 42.9 mm to (96.0, 73.0), turned to 180 degrees
- moved C9 40.2 mm to (90.2, 71.8), turned to 180 degrees
- moved C7 38.6 mm to (89.7, 68.0), turned to -90 degrees
- moved C12 35.7 mm to (99.6, 57.9), turned to 180 degrees
- moved J2 21.4 mm to (87.0, 72.0), turned to 180 degrees
- moved U4 10.9 mm to (88.8, 56.3)
Connections:
- C11 pad 2: Net-(U6-OT_PROG) -> GND
- C12 pad 2: Net-(SC2--) -> +3V3
- C9 pad 1: Net-(U5-ANT) -> +3V3
- J1 pad 1: Net-(J1-In) -> +3V3
- J2 pad 3: unconnected-(J2-~{RESET}-Pad3) -> GND
- L4 pad 1: Net-(SC2--) -> Net-(U3-DCC)
- U4 pad 1: unconnected-(U4-DEC1-Pad1) -> /LORA_RF_SW
- U4 pad 10: /LORA_BUSY -> unconnected-(U4-GND2-Pad10)
- U4 pad 11: /LORA_DIO -> /LORA_BUSY
- U4 pad 12: unconnected-(U4-VDD-Pad12) -> /LORA_DIO
- U4 pad 2: unconnected-(U4-P0.00-Pad2) -> /LORA_MISO
- U4 pad 3: unconnected-(U4-P0.01-Pad3) -> /LORA_MOSI
- U4 pad 4: /LORA_NSS -> /LORA_SCK
- U4 pad 6: /LORA_SCK -> /LORA_NSS
- U4 pad 7: /LORA_MOSI -> GND
- U4 pad 8: /LORA_MISO -> +3V3
- U4 pad 9: /LORA_RF_SW -> unconnected-(U4-ANT-Pad9)
Routing:
- net GND: track 0.00 -> 50.1 mm, vias 0 -> 10
- net /LORA_DIO: track 0.00 -> 22.4 mm
- net /LORA_BUSY: track 0.00 -> 22.3 mm
- net +3V3: track 0.00 -> 22.0 mm
- net /SWCLK: track 0.00 -> 13.9 mm
- net /LORA_RF_SW: track 0.00 -> 10.1 mm
- net /LORA_MISO: track 0.00 -> 9.71 mm
- net /LORA_NSS: track 0.00 -> 9.43 mm
- net /LORA_MOSI: track 0.00 -> 9.35 mm
- net /SWDIO: track 0.00 -> 9.27 mm
- net /LORA_NRST: track 0.00 -> 9.07 mm
- net /LORA_SCK: track 0.00 -> 8.99 mm
- net /RESET: track 0.00 -> 6.48 mm
- net Net-(U3-DCC): track 0.00 -> 3.45 mm
- net Net-(L1-Pad1): track 0.00 -> 1.82 mm
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- added copper zone on In2.Cu, net +3V3
- added copper zone on In1.Cu, net GND
Other:
- board outline added: 21 x 47 mm
