File: _autosave-nrf52.kicad_sch (KiCad schematic)
At the start: 11 parts, among them J1 Conn_ARM_JTAG_SWD_10, U1 nRF52840, U2 Wio-SX1262

Commit message: modularize
Parts:
- L2: footprint Inductor_SMD:L_0201_0603Metric -> Inductor_SMD:L_0805_2012Metric; LCSC PN C1046 -> C88173
Changed lines of the file:
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@@
 			)
 		)
-		(property "Footprint" "Inductor_SMD:L_0201_0603Metric"
+		(property "Footprint" "Inductor_SMD:L_0805_2012Metric"
 			(at 55.88 46.99 0)
 			(effects
@@
 			)
 		)
-		(property "LCSC PN" "C1046"
+		(property "LCSC PN" "C88173"
 			(at 55.88 46.99 90)
 			(effects
